File: PCB/MCU.kicad_sch (KiCad schematic)
At the start: 59 parts

Commit message: New version with FTDI chip instead of STM32 and ICE40HX FPGA instead of slower ones
Signed-off-by: Alexis Jeandet <alexis.jeandet@member.fsf.org>
Parts:
- removed J2: (no value), symbol Connector_Generic:Conn_01x06
- removed U3, U4: (no value), symbol Memory_Flash:MX25R3235FZNxx1
- C1, C10, C11, C12, C13, C14, C2, C201, C205, C206, C207, C208, C209, C211, C212, C213, C214, C215, C216, C3, C4, C5, C9: value (none) -> 100nF; footprint (none) -> Capacitor_SMD:C_0402_1005Metric
- C202, C203: value (none) -> C; footprint (none) -> Capacitor_SMD:C_0402_1005Metric
- C204, C210, C8: value (none) -> 2.2µF; footprint (none) -> Capacitor_SMD:C_1206_3216Metric_Pad1.42x1.75mm_HandSolder
- C6: renamed from C?; value (none) -> 10µF; footprint (none) -> Capacitor_SMD:C_1206_3216Metric_Pad1.42x1.75mm_HandSolder
- C7: renamed from C?; value (none) -> 100nF; footprint (none) -> Capacitor_SMD:C_0402_1005Metric
- D1, D2: value (none) -> LED; footprint (none) -> LED_SMD:LED_0603_1608Metric_Pad1.05x0.95mm_HandSolder
- J1: renamed from J?; value (none) -> USB_C_Receptacle_USB2.0; footprint (none) -> DX07S016JA1R1500:DX07S016JA1R1500
- J201: value (none) -> Conn_01x05; footprint (none) -> Connector_PinHeader_2.54mm:PinHeader_1x05_P2.54mm_Vertical
- R1, R2: value (none) -> 2.2k; footprint (none) -> Resistor_SMD:R_0402_1005Metric
- R201, R202, R203: value (none) -> 22; footprint (none) -> Resistor_SMD:R_0402_1005Metric
- R204, R205, R206, R207, R7, R8, R9: value (none) -> 100k; footprint (none) -> Resistor_SMD:R_0402_1005Metric
- R3: renamed from R?; value (none) -> 820; footprint (none) -> Resistor_SMD:R_0402_1005Metric
- R4, R5: renamed from R?; value (none) -> 5.1k; footprint (none) -> Resistor_SMD:R_0402_1005Metric
- R6: value (none) -> 3K; footprint (none) -> Resistor_SMD:R_0402_1005Metric
- SW1: value (none) -> SW_Push; footprint (none) -> Button_Switch_SMD:SW_SPST_EVQPE1
- U1: value (none) -> STM32F723ZETx; footprint (none) -> Package_QFP:LQFP-144_20x20mm_P0.5mm
- U2: value (none) -> TPD2E2U06; footprint (none) -> Package_TO_SOT_SMD:SOT-553
- U202, U203: value (none) -> TMP20AIDCK; footprint (none) -> Package_TO_SOT_SMD:SOT-353_SC-70-5
- Y201: value (none) -> 8MHz; footprint (none) -> Crystal:Resonator_SMD_muRata_CSTxExxV-3Pin_3.0x1.1mm
Connections:
- net SPI1_MISO is gone; now on net FPGA_CFG_MISO: U1.134 (PB4)
- net SPI1_MOSI is gone; now on net FPGA_CFG_MOSI: U1.135 (PB5)
- net SPI1_SCK is gone; now on net FPGA_CFG_CLK: U1.133 (PB3)
- net SPI5_NSS is gone; now on net FPGA_CFG_RESET: U1.18 (PF6)
- net SPI5_SCK is gone; now on net FPGA_CFG_DONE: U1.19 (PF7)
- net FPGA_CFG_CLK: no longer U1.111 (PC10)
- net FPGA_CFG_CS: now also U1.136 (PB6); no longer U1.40 (PA4)
- net FPGA_CFG_DONE: no longer U1.122 (PD6)
- net FPGA_CFG_MISO: no longer U1.112 (PC11)
- net FPGA_CFG_MOSI: no longer U1.113 (PC12)
- net FPGA_CFG_RESET: no longer U1.116 (PD2)
- net FPGA_HAVE_DATA: now also U1.122 (PD6); no longer U1.5 (PE6)
- net EXT_IO0: no longer names the net of U1.41 (PA5)
- net EXT_IO1: no longer names the net of U1.42 (PA6)
- net EXT_IO2: no longer names the net of U1.43 (PA7)
- net EXT_IO3: no longer names the net of U1.44 (PC4)
- net EXT_IO4: no longer names the net of U1.45 (PC5)
- net SPI1_NSS: no longer names the net of U1.110 (PA15)
- net SPI5_MISO: no longer names the net of U1.20 (PF8)
- net SPI5_MOSI: no longer names the net of U1.21 (PF9)
Other:
- note removed: "TH58CVG3S0HRAIJ"
