File: PCB/STicky.kicad_sch (KiCad schematic)
At the start: 36 parts

Commit message: New version with FTDI chip instead of STM32 and ICE40HX FPGA instead of slower ones
Signed-off-by: Alexis Jeandet <alexis.jeandet@member.fsf.org>
Parts:
- added X1: ECS-2520MV-xxx-xx, Oscillator:Oscillator_SMD_ECS_2520MV-xxx-xx-4Pin_2.5x2.0mm, symbol Oscillator:ECS-2520MV-xxx-xx
- H1, H118, H120, H2: value (none) -> MountingHole_Pad; footprint (none) -> STicky:grounding_pad_7mm
- H101, H102, H103, H104, H105, H108, H109, H110, H111, H112, H113, H116, H3, H4, H5: value (none) -> MountingHole_Pad; footprint (none) -> STicky:grounding_pad
- H106, H107, H114, H115, H117, H119: value (none) -> MountingHole_Pad; footprint (none) -> STicky:grounding_pad_9mm
- H121, H122, H123, H124, H125, H126: value (none) -> MountingHole_Pad; footprint (none) -> MountingHole:MountingHole_2.5mm_Pad
- J101, J102, J103, J104: value (none) -> Conn_Coaxial; footprint (none) -> Connector_Coaxial:SMB_Jack_Vertical
- LOGO1: value (none) -> Logo_Open_Hardware_Small; footprint (none) -> Symbol:OSHW-Logo_5.7x6mm_SilkScreen
Connections:
- net GND: now also X1.2 (GND)
- new net 12MHz: X1.3 (OUT)
- new net 3.3V: X1.1 (Tri-State), X1.4 (VDD)
Other:
- removed sheet Sheet5F66CA65
- added sheet USB (USB.kicad_sch)
- sheet Sheet5F6CBD4B ports: added FIFO_D0, FIFO_D1, FIFO_D2, FIFO_D3, FIFO_D4, FIFO_D5, FIFO_D6, FIFO_D7, FIFO_RD#, FIFO_RXF#, FIFO_SWIU, FIFO_TXE#, FIFO_WR#, OSCIN, ~{POWERDOWN}; removed FPGA_A16, FPGA_CLK, FPGA_D0, FPGA_D1, FPGA_D10, FPGA_D11, FPGA_D12, FPGA_D13, FPGA_D14, FPGA_D15, FPGA_D2, FPGA_D3, FPGA_D4, FPGA_D5, FPGA_D6, FPGA_D7, FPGA_D8, FPGA_D9, FPGA_HAVE_DATA, FPGA_NE1, FPGA_NOE, FPGA_NWE
- note removed: "MCU"

Commit message: last few fixes
Signed-off-by: Alexis Jeandet <alexis.jeandet@member.fsf.org>
Other:
- note added: "FTDI"
Changed lines of the file:
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@@
+    (effects (font (size 2.9972 2.9972) (thickness 0.5994) bold) (justify left bottom))
+  )
+  (text "FTDI" (at 73.025 83.82 0)
     (effects (font (size 2.9972 2.9972) (thickness 0.5994) bold) (justify left bottom))
   )
